File: kestrel.kicad_pcb (KiCad board)
At the start: 2 copper layers, 57.2 x 54.6 mm, 24 parts, among them J1 171971-0003, J2 171971-0003, J3 171971-0005, J4 171971-0005, J5 SBH11-PBPC-D10-ST-BK, J6 171971-0003, J7 Conn_02x02_Odd_Even, U1 MT25QXXXXXXX8EXX-XXXX, U2 MT25QXXXXXXX8EXX-XXXX, X3 PPPC202LFBN-RC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

Commit message: adapter: Update to version 1.1 with minor fixes found during testing.
- Fix signal naming for host/bmc SPI_CSb and SPI_CLK.
- Increase distance between FSI and TPM connector to allow for a shrowded TPM connector.
- Move R8/R9 (unused) to updated Csb signal locations.
- Fix silk screen for AVS1
Parts:
- moved R9 13.5 mm to (133.3, 92.7), turned to 0 degrees
- moved R8 13.0 mm to (102.9, 91.8), turned to 0 degrees
- moved J4 2.54 mm to (138.4, 64.8)
Connections:
- U1 pad 16: /flash/~HOST_SPI_CS~ -> /flash/HOST_SPI_CLK
- U1 pad 7: /flash/HOST_SPI_CLK -> /flash/~HOST_SPI_CS~
- U2 pad 16: /flash/~BMC_SPI_CS~ -> /flash/BMC_SPI_CLK
- U2 pad 7: /flash/BMC_SPI_CLK -> /flash/~BMC_SPI_CS~
- X4 pad 11: /flash/HOST_SPI_CLK -> /flash/~HOST_SPI_CS~
- X4 pad 31: /flash/~BMC_SPI_CS~ -> /flash/BMC_SPI_CLK
- X4 pad 37: /flash/BMC_SPI_CLK -> /flash/~BMC_SPI_CS~
- X4 pad 6: /flash/~HOST_SPI_CS~ -> /flash/HOST_SPI_CLK
Routing:
- net +3V3: track 134.2 -> 119.7 mm
- net /flash/~BMC_SPI_CS~: track 9.08 -> 21.4 mm
- net /flash/BMC_SPI_CLK: track 16.6 -> 6.23 mm
- net /flash/~HOST_SPI_CS~: track 12.4 -> 20.8 mm
- net /flash/HOST_SPI_CLK: track 17.1 -> 9.32 mm
- net /flash/BMC_SPI_D3: track 18.2 -> 16.1 mm
- net /flash/HOST_SPI_D3: track 20.7 -> 19.6 mm
- net /versa_expansion/FSI_DATA_EN: track 7.69 -> 8.74 mm
- net /versa_expansion/FSI_CLK: track 7.69 -> 8.74 mm
- net /versa_expansion/FSI_DATA: track 7.69 -> 8.74 mm
Other:
- board text added: "Versa Adapter v1.1"
- board text removed: "Versa Adapter v1.0"

Commit message: v1.1: Connect LPC_CLK to A12 (was PWR_LED), add pull resistor for SERIRQ.
Parts:
- added R12: 15K, Resistor_SMD:R_0603_1608Metric_Pad0.98x0.95mm_HandSolder, F.Cu at (113.0, 68.6)
- moved R2 1.27 mm to (110.5, 68.6)
- moved R6 1.27 mm to (105.4, 68.6)
- moved R3 1.27 mm to (102.9, 68.6)
- moved R4 1.27 mm to (100.3, 68.6)
- moved R5 1.27 mm to (97.8, 68.6)
- moved R7 1.27 mm to (108.0, 68.6)
Connections:
- X3 pad 5: /versa_expansion/PWD_LED -> /lpc/LPC_CLK
- X3 pad 7: Net-(X3-Pad7) -> /versa_expansion/PWD_LED
- X4 pad 3: /lpc/LPC_CLK -> Net-(X4-Pad3)
Routing:
- net /lpc/LPC_CLK: track 10.8 -> 47.5 mm
- net +3V3: track 119.7 -> 111.6 mm
- net /lpc/~LPC_SERIRQ~: track 10.8 -> 16.7 mm
- net /versa_expansion/PWD_LED: track 7.42 -> 9.79 mm
- net /versa_expansion/~PWR_BTN~: track 15.6 -> 17.3 mm
- net +3.3VP: track 19.8 -> 21.2 mm
- net /lpc/LPC_AD0: track 14.7 -> 14.2 mm
- net /lpc/LPC_AD2: track 17.2 -> 16.7 mm
- net /lpc/~LPC_RESET~: track 13.7 -> 14.2 mm
- net /lpc/~LPC_FRAME~: track 13.7 -> 14.2 mm
- net /lpc/LPC_AD3: track 13.7 -> 14.2 mm
- net /lpc/LPC_AD1: track 19.0 -> 18.5 mm
